File: 555Timer.kicad_pcb (KiCad board)
At the start: 2 copper layers, 8 parts, among them U1 NE555PWR

Commit message: changed after soproni feedback
Parts:
- moved C3 19.5 mm to (135.8, 84.5), turned to 180 degrees
Connections:
- BT1 pad 1: GND -> VCC
- BT1 pad 4: VCC -> GND
Routing:
- net VCC: track 13.8 -> 4.08 mm, vias 5 -> 0
- net GND: track 16.4 -> 15.2 mm, vias 5 -> 7

Commit message: changes
Parts:
- removed C2: 225RV0060, easyeda2kicad:CAP-SMD_BD4.0-L4.3-W4.3-LS5.0-FD
- removed RA1: CR167001F, easyeda2kicad:R0603
- added C1: VZT101M1HTR-0607, easyeda2kicad:CAP-SMD_BD6.3-L6.6-W6.6-RD, F.Cu at (125.0, 88.5)
- added R2: RC0603FR-076K8L, easyeda2kicad:R0603, F.Cu at (116.0, 103.5)
- moved RB1 0.25 mm to (115.0, 95.8), turned to -90 degrees
Routing:
- net VCC: track 4.08 -> 1.93 mm
- net Net-(U1-THRES): track 46.3 -> 45.0 mm
